Commit message: wip: steer add ackerman
Co-authored-by: Copilot <copilot@github.com>

File: src/bgr_description/urdf/bgr.urdf.xacro (robot description, xacro)
@@ -1,7 +1,4 @@
 <?xml version="1.0"?>
 <robot name="bgr" xmlns:xacro="http://ros.org/wiki/xacro">
-  <!-- External includes-->
-  <xacro:include filename="$(find bgr_description)/urdf/bgr_gazebo.xacro"/>
-  <xacro:include filename="$(find bgr_description)/urdf/bgr_ros2_control.xacro"/>
   <!-- === Basic params === -->
   <!-- Wheel geometry (radius/width) and chassis dimensions -->
@@ -12,10 +9,30 @@
   <xacro:property name="wheelbase"    value="2.0368"/>
    <!-- Mass and steering limits -->
-  <xacro:property name="body_mass"    value="50.0"/>
+  <!-- Real measured total car mass is 283.6 kg. body_mass is the remaining
+       base_link mass after separately modeled wheels, steering stubs, and sensors. -->
+  <xacro:property name="total_vehicle_mass" value="283.6"/>
+  <xacro:property name="wheel_mass"         value="5.0"/>
+  <xacro:property name="steering_stub_mass" value="0.01"/>
+  <xacro:property name="lidar_mass"         value="0.5"/>
+  <xacro:property name="imu_mass"           value="0.1"/>
+  <xacro:property name="front_cam_mass"     value="0.01"/>
+  <xacro:property name="body_mass"          value="${total_vehicle_mass - (4*wheel_mass + 2*steering_stub_mass + lidar_mass + imu_mass + front_cam_mass)}"/>
+  <xacro:property name="wheel_normal_force" value="${total_vehicle_mass * 9.80665 / 4.0}"/>
   <xacro:property name="steer_limit"  value="0.6"/>
-  <!-- Bounding box used for base_link collision and inertia -->
-  <xacro:property name="body_size_x"  value="2.0"/>
-  <xacro:property name="body_size_y"  value="1.0"/>
-  <xacro:property name="body_size_z"  value="0.5"/>
+  <!-- Mesh-bounds approximation used for base_link collision and inertia.
+       Replace body_cg_* with measured CG values when available. -->
+  <xacro:property name="body_size_x"             value="3.140043"/>
+  <xacro:property name="body_size_y"             value="1.606011"/>
+  <xacro:property name="body_size_z"             value="1.151132"/>
+  <xacro:property name="body_collision_origin_x" value="0.074010"/>
+  <xacro:property name="body_collision_origin_y" value="0.0"/>
+  <xacro:property name="body_collision_origin_z" value="0.153035"/>
+  <xacro:property name="body_cg_x"               value="${body_collision_origin_x}"/>
+  <xacro:property name="body_cg_y"               value="${body_collision_origin_y}"/>
+  <xacro:property name="body_cg_z"               value="${body_collision_origin_z}"/>
+  <!-- External includes. Keep these after shared properties so Gazebo and
+       ros2_control fragments can reuse the same physical dimensions. -->
+  <xacro:include filename="$(find bgr_description)/urdf/bgr_gazebo.xacro"/>
+  <xacro:include filename="$(find bgr_description)/urdf/bgr_ros2_control.xacro"/>
   <!-- === Base footprint === -->
   <link name="base_footprint"/>
@@ -29,5 +46,5 @@
     <!-- Box inertia -->
     <inertial>
-      <origin xyz="0 0 0" rpy="0 0 0"/>
+      <origin xyz="${body_cg_x} ${body_cg_y} ${body_cg_z}" rpy="0 0 0"/>
       <mass value="${body_mass}"/>
       <inertia ixx="${1.0/12.0*body_mass*(body_size_y*body_size_y + body_size_z*body_size_z)}"
@@ -46,5 +63,5 @@
     <!-- Collision as box (affects physics) -->
     <collision>
-      <origin xyz="0 0 ${body_size_z/2}" rpy="0 0 0"/>
+      <origin xyz="${body_collision_origin_x} ${body_collision_origin_y} ${body_collision_origin_z}" rpy="0 0 0"/>
       <geometry>
         <box size="${body_size_x} ${body_size_y} ${body_size_z}"/>
@@ -57,8 +74,8 @@
       <inertial>
         <origin xyz="0 0 0" rpy="0 0 0"/>
-        <mass value="5.0"/>
-        <inertia ixx="${(1.0/12.0)*5.0*(3*wheel_radius*wheel_radius + wheel_width*wheel_width)}"
-                 iyy="${(1.0/12.0)*5.0*(3*wheel_radius*wheel_radius + wheel_width*wheel_width)}"
-                 izz="${0.5*5.0*wheel_radius*wheel_radius}"
+        <mass value="${wheel_mass}"/>
+        <inertia ixx="${(1.0/12.0)*wheel_mass*(3*wheel_radius*wheel_radius + wheel_width*wheel_width)}"
+                 iyy="${0.5*wheel_mass*wheel_radius*wheel_radius}"
+                 izz="${(1.0/12.0)*wheel_mass*(3*wheel_radius*wheel_radius + wheel_width*wheel_width)}"
                  ixy="0" ixz="0" iyz="0"/>
       </inertial>
@@ -84,5 +101,5 @@
     <link name="${name}">
       <inertial>
-        <mass value="0.01"/>
+        <mass value="${steering_stub_mass}"/>
         <origin xyz="0 0 0" rpy="0 0 0"/>
         <inertia ixx="1e-5" ixy="0" ixz="0" iyy="1e-5" iyz="0" izz="1e-5"/>
@@ -130,5 +147,4 @@
     <limit lower="${-steer_limit}" upper="${steer_limit}" effort="200" velocity="2.0"/>
     <dynamics damping="1.5" friction="0.1"/>
-    <mimic joint="Steering_fr_joint" multiplier="1.0" offset="0.0"/>
   </joint>
   <!-- left front wheel -->
@@ -167,5 +183,5 @@
   <link name="lidar_link">
     <inertial>
-      <mass value="0.5"/>
+      <mass value="${lidar_mass}"/>
       <origin xyz="0 0 0" rpy="0 0 0"/>
       <inertia ixx="0.001" ixy="0" ixz="0" iyy="0.001" iyz="0" izz="0.001"/>
@@ -193,5 +209,5 @@
   <link name="imu_link">
     <inertial>
-      <mass value="0.1"/>
+      <mass value="${imu_mass}"/>
       <origin xyz="0 0 0" rpy="0 0 0"/>
       <inertia ixx="0.00001" ixy="0" ixz="0" iyy="0.00001" iyz="0" izz="0.00001"/>
@@ -202,5 +218,5 @@
     <inertial>
       <origin xyz="0 0 0" rpy="0 0 0"/>
-      <mass value="0.01"/>
+      <mass value="${front_cam_mass}"/>
       <inertia ixx="0.001" ixy="0" ixz="0" iyy="0.001" iyz="0" izz="0.001"/>
     </inertial>

File: src/bgr_description/urdf/bgr_gazebo.xacro (robot description, xacro)
@@ -57,22 +57,29 @@
     </plugin>
   </gazebo>
-  <!-- Note: Steering mimic handling in Gazebo Harmonic dart is not natively supported
-       via the gz-sim-mimic-joint-system plugin. It relies on ros2_control to enforce it. -->
+  <!-- Steering is commanded as independent Ackermann left/right joint positions via ros2_control. -->
   <!-- Wheel slip plugin for better rolling behavior (all wheels) -->
   <gazebo>
     <plugin filename="gz-sim-wheel-slip-system" name="gz::sim::systems::WheelSlip">
       <wheel link_name="Wheel_rr">
+        <wheel_radius>${wheel_radius}</wheel_radius>
+        <wheel_normal_force>${wheel_normal_force}</wheel_normal_force>
         <slip_compliance_lateral>0.05</slip_compliance_lateral>
         <slip_compliance_longitudinal>0.001</slip_compliance_longitudinal>
       </wheel>
       <wheel link_name="Wheel_rl">
+        <wheel_radius>${wheel_radius}</wheel_radius>
+        <wheel_normal_force>${wheel_normal_force}</wheel_normal_force>
         <slip_compliance_lateral>0.05</slip_compliance_lateral>
         <slip_compliance_longitudinal>0.001</slip_compliance_longitudinal>
       </wheel>
       <wheel link_name="Wheel_fr">
+        <wheel_radius>${wheel_radius}</wheel_radius>
+        <wheel_normal_force>${wheel_normal_force}</wheel_normal_force>
         <slip_compliance_lateral>0.05</slip_compliance_lateral>
         <slip_compliance_longitudinal>0.001</slip_compliance_longitudinal>
       </wheel>
       <wheel link_name="Wheel_fl">
+        <wheel_radius>${wheel_radius}</wheel_radius>
+        <wheel_normal_force>${wheel_normal_force}</wheel_normal_force>
         <slip_compliance_lateral>0.05</slip_compliance_lateral>
         <slip_compliance_longitudinal>0.001</slip_compliance_longitudinal>

File: src/bgr_description/urdf/bgr_ros2_control.xacro (robot description, xacro)
@@ -25,15 +25,18 @@
         <!-- Front steering and wheels -->
         <joint name="Steering_fl_joint">
-        <!-- Mimic joint: expose only state interfaces (no commands) -->
-        <state_interface name="position"/>
-        <state_interface name="velocity"/>
+            <command_interface name="position">
+                <param name="min">-0.6</param>
+                <param name="max">0.6</param>
+            </command_interface>
+            <state_interface name="position"/>
+            <state_interface name="velocity"/>
         </joint>
         <joint name="Steering_fr_joint">
-        <command_interface name="position">
-            <param name="min">-1</param>
-            <param name="max">1</param>
-        </command_interface>
-        <state_interface name="position"/>
-        <state_interface name="velocity"/>
+            <command_interface name="position">
+                <param name="min">-0.6</param>
+                <param name="max">0.6</param>
+            </command_interface>
+            <state_interface name="position"/>
+            <state_interface name="velocity"/>
         </joint>
          <!-- Front wheels: velocity-controlled by controllers -->
