Commit message: Update file paths and add lidar support in URDF and SDF configurations

File: src/bgr_description/urdf/bgr.urdf.xacro (robot description, xacro)
@@ -20,4 +20,11 @@
   <xacro:property name="body_size_y"  value="1.0"/>
   <xacro:property name="body_size_z"  value="0.5"/>
+  <!-- === Base footprint === -->
+  <link name="base_footprint"/>
+  <joint name="base_joint" type="fixed">
+    <parent link="base_footprint"/>
+    <child link="base_link"/>
+    <origin xyz="0 0 0" rpy="0 0 0"/>
+  </joint>
    <!--  Base link (chassis) -->
   <link name="base_link">
@@ -154,3 +161,29 @@
     <dynamics damping="0.03" friction="0.01"/>
   </joint>
+  <!-- Lidar -->
+  <joint name="lidar_joint" type="fixed">
+    <origin xyz="0.5 0 0.3" rpy="0 0 0"/>
+    <parent link="base_link"/>
+    <child link="lidar_link"/>
+  </joint>
+  <link name="lidar_link">
+    <inertial>
+      <mass value="0.5"/>
+      <origin xyz="0 0 0" rpy="0 0 0"/>
+      <inertia ixx="0.001" ixy="0" ixz="0" iyy="0.001" iyz="0" izz="0.001"/>
+    </inertial>
+    <visual>
+      <geometry>
+        <cylinder radius="0.05" length="0.05"/>
+      </geometry>
+      <material name="black">
+        <color rgba="0 0 0 1"/>
+      </material>
+    </visual>
+    <collision>
+      <geometry>
+        <cylinder radius="0.05" length="0.05"/>
+      </geometry>
+    </collision>
+  </link>
 </robot>

File: src/bgr_description/urdf/bgr_gazebo.xacro (robot description, xacro)
@@ -104,3 +104,36 @@
     </xacro:unless>
   </gazebo>
+<!-- Lidar -->
+  <gazebo reference="lidar_link">
+    <sensor name="lidar" type="gpu_lidar"> <topic>scan</topic> <!-- if there is a gpu - switch type="lidar"> to type="gpu_lidar" -->
+      <pose>0 0 0 0 0 0</pose>
+      <always_on>true</always_on>
+      <visualize>true</visualize>
+      <update_rate>10</update_rate>
+      <ray>
+         <scan>
+            <horizontal>
+              <samples>360</samples>
+              <resolution>1</resolution>
+              <min_angle>-3.14159</min_angle>
+              <max_angle>3.14159</max_angle>
+            </horizontal>
+            <vertical>
+            <samples>32</samples>
+            <resolution>1</resolution>
+            <min_angle>-0.26</min_angle> <max_angle>0.26</max_angle>  </vertical>
+          </scan>
+          <range>
+            <min>0.10</min>
+            <max>30.0</max>
+            <resolution>0.01</resolution>
+          </range>
+      </ray>
+    </sensor>
+  </gazebo>
+  <gazebo>
+    <plugin filename="libgz-sim-sensors-system" name="gz::sim::systems::Sensors">
+      <render_engine>ogre2</render_engine>
+    </plugin>
+  </gazebo>
 </robot>

Commit message: Cam Sens integrated with main

File: src/bgr_description/urdf/bgr.urdf.xacro (robot description, xacro)
@@ -187,3 +187,23 @@
     </collision>
   </link>
+  <!-- Chase Camera -->
+  <link name="chase_cam_link">
+    <inertial>
+      <mass value="0.01"/>
+      <inertia ixx="0.001" ixy="0" ixz="0" iyy="0.001" iyz="0" izz="0.001"/>
+    </inertial>
+    <visual>
+      <geometry>
+        <box size="0.05 0.05 0.05"/>
+      </geometry>
+      <material name="blue">
+        <color rgba="0 0 1 1"/>
+      </material>
+    </visual>
+  </link>
+  <joint name="chase_cam_joint" type="fixed">
+    <parent link="base_link"/>
+    <child link="chase_cam_link"/>
+    <origin xyz="0.5 0 0.38" rpy="0 0 0"/>
+  </joint>
 </robot>

File: src/bgr_description/urdf/bgr_gazebo.xacro (robot description, xacro)
@@ -133,8 +133,41 @@
     </sensor>
   </gazebo>
-  <gazebo>
+  <!-- <gazebo>
     <plugin filename="gz-sim-sensors-system" name="gz::sim::systems::Sensors">
       <render_engine>ogre2</render_engine>
     </plugin>
+  </gazebo> -->
+  <gazebo reference="chase_cam_link">
+    <sensor name="chase_camera" type="camera">
+      <pose>0 0 0 0 0 0</pose>
+      <visualize>true</visualize>
+      <update_rate>30</update_rate>
+      <topic>chase_cam</topic>
+      <camera>
+        <horizontal_fov>1.2</horizontal_fov>
+        <image>
+          <width>800</width>
+          <height>600</height>
+          <format>R8G8B8</format>
+        </image>
+        <clip>
+          <near>0.1</near>
+          <far>1000</far>
+        </clip>
+      </camera>
+    </sensor>
+  </gazebo>
+  <!-- Correct sensor plugin varying by ros version-->
+  <gazebo>
+    <xacro:if value="$(arg is_ignition)">
+      <plugin filename="ign-gazebo-sensors-system" name="ignition::gazebo::systems::Sensors">
+        <render_engine>ogre2</render_engine>
+      </plugin>
+    </xacro:if>
+    <xacro:unless value="$(arg is_ignition)">
+      <plugin filename="gz-sim-sensors-system" name="gz::sim::systems::Sensors">
+        <render_engine>ogre2</render_engine>
+      </plugin>
+    </xacro:unless>
   </gazebo>
 </robot>

Commit message: Changed chase_cam name to front_cam, working camera sensor

File: src/bgr_description/urdf/bgr.urdf.xacro (robot description, xacro)
@@ -187,6 +187,6 @@
     </collision>
   </link>
-  <!-- Chase Camera -->
-  <link name="chase_cam_link">
+  <!-- Front Camera - To run: ros2 run rqt_image_view rqt_image_view after launching gazebo -->
+  <link name="front_cam_link">
     <inertial>
       <mass value="0.01"/>
@@ -202,7 +202,7 @@
     </visual>
   </link>
-  <joint name="chase_cam_joint" type="fixed">
-    <parent link="base_link"/>
-    <child link="chase_cam_link"/>
+  <joint name="front_cam_joint" type="fixed">
+    <parent link="base_link"/>
+    <child link="front_cam_link"/>
     <origin xyz="0.5 0 0.38" rpy="0 0 0"/>
   </joint>

File: src/bgr_description/urdf/bgr_gazebo.xacro (robot description, xacro)
@@ -138,10 +138,11 @@
     </plugin>
   </gazebo> -->
-  <gazebo reference="chase_cam_link">
-    <sensor name="chase_camera" type="camera">
+  <!-- Front Camera -->
+  <gazebo reference="front_cam_link">
+    <sensor name="front_camera" type="camera">
       <pose>0 0 0 0 0 0</pose>
       <visualize>true</visualize>
       <update_rate>30</update_rate>
-      <topic>chase_cam</topic>
+      <topic>front_cam</topic>
       <camera>
         <horizontal_fov>1.2</horizontal_fov>
