Commit message: Add motor controller and update controller configurations for effort control

File: src/bgr_description/urdf/bgr.urdf.xacro (robot description, xacro)
@@ -1,58 +1,44 @@
 <?xml version="1.0"?>
 <robot name="bgr" xmlns:xacro="http://ros.org/wiki/xacro">
-   <!-- Select Gazebo flavor (Ignition/GZ) to load the matching ros2_control hardware plugin -->
   <xacro:arg name="is_ignition" default="true"/>
-  <!-- External includes-->
   <xacro:include filename="$(find bgr_description)/urdf/bgr_gazebo.xacro"/>
   <xacro:include filename="$(find bgr_description)/urdf/bgr_ros2_control.xacro"/>
-  <!-- === Basic params === -->
-  <!-- Wheel geometry (radius/width) and chassis dimensions -->
   <xacro:property name="wheel_radius" value="0.24"/>
   <xacro:property name="wheel_width"  value="0.12"/>
-  <!-- Track = left-right distance between wheel centers; Wheelbase = front-rear distance -->
-  <xacro:property name="track"        value="1.3092"/>
-  <xacro:property name="wheelbase"    value="2.0368"/>
-   <!-- Mass and steering limits -->
-  <xacro:property name="body_mass"    value="50.0"/>
-  <xacro:property name="steer_limit"  value="0.6"/>
-  <!-- Bounding box used for base_link collision and inertia -->
+  <xacro:property name="track"         value="1.3092"/>
+  <xacro:property name="wheelbase"     value="2.0368"/>
+  <xacro:property name="body_mass"     value="286.0"/>
+  <xacro:property name="steer_limit"  value="0.384"/>
+  <xacro:property name="motor_inertia_kgm2" value="0.000274"/>
+  <xacro:property name="gear_ratio"           value="11.5"/>
+  <xacro:property name="reflected_inertia"    value="${motor_inertia_kgm2 * gear_ratio * gear_ratio}"/>
+  <xacro:property name="ixx_val"  value="55.801289"/>
+  <xacro:property name="iyy_val"  value="181.382241"/>
+  <xacro:property name="izz_val"  value="199.609647"/>
+  <xacro:property name="ixy_val"  value="-0.288597"/>
+  <xacro:property name="ixz_val"  value="-8.267511"/>
+  <xacro:property name="iyz_val"  value="-0.015345"/>
   <xacro:property name="body_size_x"  value="2.0"/>
   <xacro:property name="body_size_y"  value="1.0"/>
   <xacro:property name="body_size_z"  value="0.5"/>
-  <!-- === Base footprint === -->
-  <link name="base_footprint"/>
-  <joint name="base_joint" type="fixed">
-    <parent link="base_footprint"/>
-    <child link="base_link"/>
-    <origin xyz="0 0 0" rpy="0 0 0"/>
-  </joint>
-   <!--  Base link (chassis) -->
   <link name="base_link">
-    <!-- Box inertia -->
     <inertial>
       <origin xyz="0 0 0" rpy="0 0 0"/>
       <mass value="${body_mass}"/>
-      <inertia ixx="${1.0/12.0*body_mass*(body_size_y*body_size_y + body_size_z*body_size_z)}"
-               iyy="${1.0/12.0*body_mass*(body_size_x*body_size_x + body_size_z*body_size_z)}"
-               izz="${1.0/12.0*body_mass*(body_size_x*body_size_x + body_size_y*body_size_y)}"
-               ixy="0" ixz="0" iyz="0"/>
+      <inertia ixx="${ixx_val}" iyy="${iyy_val}" izz="${izz_val}"
+               ixy="${ixy_val}" ixz="${ixz_val}" iyz="${iyz_val}"/>
     </inertial>
-    <!-- Visual STL File (doesn't affect physics) -->
     <visual>
       <origin xyz="0 0 0" rpy="0 0 0"/>
-      <geometry>
-        <mesh filename="package://bgr_description/meshes/visual/base_link.STL"/>
-      </geometry>
-      <material name=""><color rgba="0.79216 0.81961 0.93333 1"/></material>
+      <geometry><mesh filename="package://bgr_description/meshes/visual/base_link.STL"/></geometry>
+      <material name="blue_grey">
+          <color rgba="0.79216 0.81961 0.93333 1"/>
+      </material>
     </visual>
-    <!-- Collision as box (affects physics) -->
     <collision>
       <origin xyz="0 0 ${body_size_z/2}" rpy="0 0 0"/>
-      <geometry>
-        <box size="${body_size_x} ${body_size_y} ${body_size_z}"/>
-      </geometry>
+      <geometry><box size="${body_size_x} ${body_size_y} ${body_size_z}"/></geometry>
     </collision>
   </link>
-  <!-- === Wheel link macro === -->
   <xacro:macro name="wheel_link" params="name visual_mesh">
     <link name="${name}">
@@ -60,27 +46,23 @@
         <origin xyz="0 0 0" rpy="0 0 0"/>
         <mass value="5.0"/>
-        <inertia ixx="${(1.0/12.0)*5.0*(3*wheel_radius*wheel_radius + wheel_width*wheel_width)}"
-                 iyy="${(1.0/12.0)*5.0*(3*wheel_radius*wheel_radius + wheel_width*wheel_width)}"
-                 izz="${0.5*5.0*wheel_radius*wheel_radius}"
-                 ixy="0" ixz="0" iyz="0"/>
+        <inertia
+          ixx="${(1.0/12.0)*5.0*(3*wheel_radius*wheel_radius + wheel_width*wheel_width) + reflected_inertia}"
+          iyy="${(1.0/12.0)*5.0*(3*wheel_radius*wheel_radius + wheel_width*wheel_width) + reflected_inertia}"
+          izz="${(0.5*5.0*wheel_radius*wheel_radius) + reflected_inertia}"
+          ixy="0" ixz="0" iyz="0"/>
       </inertial>
-      <!-- Visual mesh -->
       <visual>
         <origin xyz="0 0 0" rpy="0 0 0"/>
-        <geometry>
-          <mesh filename="${visual_mesh}"/>
-        </geometry>
-        <material name=""><color rgba="0.79216 0.81961 0.93333 1"/></material>
+        <geometry><mesh filename="${visual_mesh}"/></geometry>
+        <material name="blue_grey">
+            <color rgba="0.79216 0.81961 0.93333 1"/>
+        </material>
       </visual>
-      <!-- Collision as cylinder -->
       <collision>
         <origin xyz="0 0 0" rpy="1.57079632679 0 0"/>
-        <geometry>
-          <cylinder radius="${wheel_radius}" length="${wheel_width}"/>
-        </geometry>
+        <geometry><cylinder radius="${wheel_radius}" length="${wheel_width}"/></geometry>
       </collision>
     </link>
   </xacro:macro>
-  <!-- === Stub link macro (for steering knuckles) === -->
   <xacro:macro name="stub_link" params="name">
     <link name="${name}">
@@ -96,94 +78,45 @@
     </link>
   </xacro:macro>
-  <!-- === Wheels and Joints === -->
-  <!-- rear wheels -->
   <xacro:wheel_link name="Wheel_rl" visual_mesh="package://bgr_description/meshes/visual/Wheel_rl.STL"/>
   <xacro:wheel_link name="Wheel_rr" visual_mesh="package://bgr_description/meshes/visual/Wheel_rr.STL"/>
-  <!-- front wheels with steering stubs -->
   <xacro:stub_link name="Steering_fl"/>
   <xacro:wheel_link name="Wheel_fl" visual_mesh="package://bgr_description/meshes/visual/Wheel_fl.STL"/>
   <xacro:stub_link name="Steering_fr"/>
   <xacro:wheel_link name="Wheel_fr" visual_mesh="package://bgr_description/meshes/visual/Wheel_fr.STL"/>
-  <!-- === Joints === -->
-  <!-- rear left -->
   <joint name="Wheel_rl_joint" type="continuous">
-    <origin xyz="${-wheelbase/2} ${ track/2} -${wheel_radius}" rpy="0 0 0"/>
-    <parent link="base_link"/>
-    <child  link="Wheel_rl"/>
-    <axis xyz="0 1 0"/>
-    <limit effort="200" velocity="100"/>
-    <dynamics damping="0.05" friction="0.01"/>
+    <origin xyz="${-wheelbase/2} ${track/2} -${wheel_radius}" rpy="0 0 0"/>
+    <parent link="base_link"/><child link="Wheel_rl"/><axis xyz="0 1 0"/>
+    <limit effort="300" velocity="100"/>
+    <dynamics damping="1.0" friction="1.0"/>
   </joint>
-  <!-- rear right -->
   <joint name="Wheel_rr_joint" type="continuous">
     <origin xyz="${-wheelbase/2} ${-track/2} -${wheel_radius}" rpy="0 0 0"/>
-    <parent link="base_link"/>
-    <child  link="Wheel_rr"/>
-    <axis xyz="0 1 0"/>
-    <limit effort="200" velocity="100"/>
-    <dynamics damping="0.05" friction="0.01"/>
+    <parent link="base_link"/><child link="Wheel_rr"/><axis xyz="0 1 0"/>
+    <limit effort="300" velocity="100"/>
+    <dynamics damping="1.0" friction="1.0"/>
   </joint>
-  <!-- steering front left-->
   <joint name="Steering_fl_joint" type="revolute">
-    <origin xyz="${ wheelbase/2} ${ track/2} -${wheel_radius}" rpy="0 0 0"/>
-    <parent link="base_link"/>
-    <child  link="Steering_fl"/>
-    <axis xyz="0 0 1"/>
-    <limit lower="${-steer_limit}" upper="${steer_limit}" effort="200" velocity="2.0"/>
-    <dynamics damping="1.5" friction="0.1"/>
-    <mimic joint="Steering_fr_joint" multiplier="1.0" offset="0.0"/>
-  </joint>
-  <!-- left front wheel -->
-  <joint name="Wheel_fl_joint" type="continuous">
-    <origin xyz="0 0 0" rpy="0 0 0"/>
-    <parent link="Steering_fl"/>
-    <child  link="Wheel_fl"/>
-    <axis xyz="0 1 0"/>
-    <limit effort="200" velocity="100"/>
-    <dynamics damping="0.03" friction="0.01"/>
-  </joint>
-  <!-- steering front right-->
-  <joint name="Steering_fr_joint" type="revolute">
-    <origin xyz="${ wheelbase/2} ${-track/2} -${wheel_radius}" rpy="0 0 0"/>
-    <parent link="base_link"/>
-    <child  link="Steering_fr"/>
-    <axis xyz="0 0 1"/>
+    <origin xyz="${wheelbase/2} ${track/2} -${wheel_radius}" rpy="0 0 0"/>
+    <parent link="base_link"/><child link="Steering_fl"/><axis xyz="0 0 1"/>
     <limit lower="${-steer_limit}" upper="${steer_limit}" effort="200" velocity="2.0"/>
     <dynamics damping="1.5" friction="0.1"/>
   </joint>
-  <!-- right front wheel -->
+  <joint name="Wheel_fl_joint" type="continuous">
+    <origin xyz="0 0 0" rpy="0 0 0"/>
+    <parent link="Steering_fl"/><child link="Wheel_fl"/><axis xyz="0 1 0"/>
+    <limit effort="300" velocity="100"/>
+    <dynamics damping="1.0" friction="1.0"/>
+  </joint>
+  <joint name="Steering_fr_joint" type="revolute">
+    <origin xyz="${wheelbase/2} ${-track/2} -${wheel_radius}" rpy="0 0 0"/>
+    <parent link="base_link"/><child link="Steering_fr"/><axis xyz="0 0 1"/>
+    <limit lower="${-steer_limit}" upper="${steer_limit}" effort="200" velocity="2.0"/>
+    <dynamics damping="1.5" friction="0.1"/>
+  </joint>
   <joint name="Wheel_fr_joint" type="continuous">
     <origin xyz="0 0 0" rpy="0 0 0"/>
-    <parent link="Steering_fr"/>
-    <child  link="Wheel_fr"/>
-    <axis xyz="0 1 0"/>
-    <limit effort="200" velocity="100"/>
-    <dynamics damping="0.03" friction="0.01"/>
+    <parent link="Steering_fr"/><child link="Wheel_fr"/><axis xyz="0 1 0"/>
+    <limit effort="300" velocity="100"/>
+    <dynamics damping="1.0" friction="1.0"/>
   </joint>
-  <!-- Lidar -->
-  <joint name="lidar_joint" type="fixed">
-    <origin xyz="0.5 0 0.3" rpy="0 0 0"/>
-    <parent link="base_link"/>
-    <child link="lidar_link"/>
-  </joint>
-  <link name="lidar_link">
-    <inertial>
-      <mass value="0.5"/>
-      <origin xyz="0 0 0" rpy="0 0 0"/>
-      <inertia ixx="0.001" ixy="0" ixz="0" iyy="0.001" iyz="0" izz="0.001"/>
-    </inertial>
-    <visual>
-      <geometry>
-        <cylinder radius="0.05" length="0.05"/>
-      </geometry>
-      <material name="black">
-        <color rgba="0 0 0 1"/>
-      </material>
-    </visual>
-    <collision>
-      <geometry>
-        <cylinder radius="0.05" length="0.05"/>
-      </geometry>
-    </collision>
-  </link>
 </robot>

File: src/bgr_description/urdf/bgr_gazebo.xacro (robot description, xacro)
@@ -1,40 +1,19 @@
 <?xml version="1.0"?>
 <robot name="bgr" xmlns:xacro="http://ros.org/wiki/xacro">
-  <!-- Gazebo specific parameters -->
-  <gazebo reference="Wheel_fl">
-    <mu1>1.2</mu1><mu2>1.2</mu2> <!-- coefficient of friction -->
-    <surface>
-      <friction><ode><mu>1.2</mu><mu2>1.2</mu2><slip1>0.01</slip1><slip2>0.01</slip2></ode></friction> <!-- friction parameters -->
-      <contact><ode><kp>1000000.0</kp><kd>1.0</kd><max_vel>0.1</max_vel><min_depth>0.001</min_depth></ode></contact> <!-- contact parameters -->
-    </surface>
-  </gazebo>
-  <gazebo reference="Wheel_fr">
-    <mu1>1.2</mu1><mu2>1.2</mu2>
-    <surface>
-      <friction><ode><mu>1.2</mu><mu2>1.2</mu2><slip1>0.01</slip1><slip2>0.01</slip2></ode></friction>
-      <contact><ode><kp>1000000.0</kp><kd>1.0</kd><max_vel>0.1</max_vel><min_depth>0.001</min_depth></ode></contact>
-    </surface>
-  </gazebo>
-  <gazebo reference="Wheel_rl">
-    <mu1>1.2</mu1><mu2>1.2</mu2>
-    <surface>
-      <friction><ode><mu>1.2</mu><mu2>1.2</mu2><slip1>0.01</slip1><slip2>0.01</slip2></ode></friction>
-      <contact><ode><kp>1000000.0</kp><kd>1.0</kd><max_vel>0.1</max_vel><min_depth>0.001</min_depth></ode></contact>
-    </surface>
-  </gazebo>
-  <gazebo reference="Wheel_rr">
-    <mu1>1.2</mu1><mu2>1.2</mu2>
-    <surface>
-      <friction><ode><mu>1.2</mu><mu2>1.2</mu2><slip1>0.01</slip1><slip2>0.01</slip2></ode></friction>
-      <contact><ode><kp>1000000.0</kp><kd>1.0</kd><max_vel>0.1</max_vel><min_depth>0.001</min_depth></ode></contact>
-    </surface>
-  </gazebo>
-  <!-- Chassis friction -->
-  <gazebo reference="base_link">
-    <mu1>0.2</mu1><mu2>0.2</mu2>
-  </gazebo>
-  <!-- ROS 2 Control -->
+  <xacro:macro name="wheel_gazebo_ref" params="reference">
+    <gazebo reference="${reference}">
+      <mu1>1.5</mu1>
+      <mu2>1.5</mu2>
+      <kp>1000000.0</kp>
+      <kd>10.0</kd>
+      <minDepth>0.001</minDepth>
+      <maxVel>0.1</maxVel>
+    </gazebo>
+  </xacro:macro>
+  <xacro:wheel_gazebo_ref reference="Wheel_fl"/>
+  <xacro:wheel_gazebo_ref reference="Wheel_fr"/>
+  <xacro:wheel_gazebo_ref reference="Wheel_rl"/>
+  <xacro:wheel_gazebo_ref reference="Wheel_rr"/>
   <gazebo>
-    <!-- ROS 2 Humble -->
     <xacro:if value="$(arg is_ignition)">
       <plugin filename="ign_ros2_control-system" name="ign_ros2_control::IgnitionROS2ControlPlugin">
@@ -42,5 +21,4 @@
       </plugin>
     </xacro:if>
-    <!-- ROS 2 Iron or above -->
     <xacro:unless value="$(arg is_ignition)">
       <plugin filename="gz_ros2_control-system" name="gz_ros2_control::GazeboSimROS2ControlPlugin">
@@ -49,5 +27,4 @@
     </xacro:unless>
   </gazebo>
-  <!-- Publishes /joint_states for all defined joints -->
   <gazebo>
     <plugin filename="gz-sim-joint-state-publisher-system" name="gz::sim::systems::JointStatePublisher">
@@ -61,79 +38,9 @@
     </plugin>
   </gazebo>
-  <!-- Enforce steering mimic in physics (FL follows FR) -->
   <gazebo>
-    <plugin filename="gz-sim-mimic-joint-system" name="gz::sim::systems::MimicJoint">
-      <joint_name>Steering_fl_joint</joint_name>
-      <mimicked_joint>Steering_fr_joint</mimicked_joint>
-      <multiplier>-1.0</multiplier>
-      <offset>0.0</offset>
-    </plugin>
-  </gazebo>
-  <!-- Wheel slip plugin for better rolling behavior (all wheels) -->
-  <gazebo>
-    <plugin filename="gz-sim-wheel-slip-system" name="gz::sim::systems::WheelSlip">
-      <wheel link_name="Wheel_rr">
-        <slip_compliance_lateral>0.05</slip_compliance_lateral>
-        <slip_compliance_longitudinal>0.001</slip_compliance_longitudinal>
-      </wheel>
-      <wheel link_name="Wheel_rl">
-        <slip_compliance_lateral>0.05</slip_compliance_lateral>
-        <slip_compliance_longitudinal>0.001</slip_compliance_longitudinal>
-      </wheel>
-      <wheel link_name="Wheel_fr">
-        <slip_compliance_lateral>0.05</slip_compliance_lateral>
-        <slip_compliance_longitudinal>0.001</slip_compliance_longitudinal>
-      </wheel>
-      <wheel link_name="Wheel_fl">
-        <slip_compliance_lateral>0.05</slip_compliance_lateral>
-        <slip_compliance_longitudinal>0.001</slip_compliance_longitudinal>
-      </wheel>
-    </plugin>
-  </gazebo>
-    <!-- Publish ground-truth pose of the BGR car as /model/bgr/pose in Gazebo -->
-  <!-- GROUND TRUTH ODOMETRY (Perfect Position) -->
-  <gazebo>
-    <xacro:unless value="$(arg is_ignition)">
-      <plugin filename="gz-sim-odometry-publisher-system"
-              name="gz::sim::systems::OdometryPublisher">
-        <dimensions>3</dimensions> <!-- 3D Position -->
-        <odom_frame>world</odom_frame> <!-- Calculate relative to the World -->
-        <robot_base_frame>base_link</robot_base_frame>
-        <odom_publish_frequency>50</odom_publish_frequency>
-      </plugin>
-    </xacro:unless>
-  </gazebo>
-<!-- Lidar -->
-  <gazebo reference="lidar_link">
-    <sensor name="lidar" type="gpu_lidar">
-      <topic>lidar</topic>
-      <pose>0 0 0 0 0 0</pose>
-      <always_on>true</always_on>
-      <visualize>true</visualize>
-      <update_rate>10</update_rate>
-      <ray>
-         <scan>
-            <horizontal>
-              <samples>360</samples>
-              <resolution>1</resolution>
-              <min_angle>-1</min_angle>
-              <max_angle>1</max_angle>
-            </horizontal>
-            <vertical>
-            <samples>256</samples>
-            <resolution>1</resolution>
-            <min_angle>-0.218</min_angle> <max_angle>0.218</max_angle>  </vertical>
-          </scan>
-          <range>
-            <min>0.10</min>
-            <max>30.0</max>
-            <resolution>0.01</resolution>
-          </range>
-      </ray>
-    </sensor>
-  </gazebo>
-  <gazebo>
-    <plugin filename="gz-sim-sensors-system" name="gz::sim::systems::Sensors">
-      <render_engine>ogre2</render_engine>
+    <plugin filename="gz-sim-odometry-publisher-system" name="gz::sim::systems::OdometryPublisher">
+      <odom_frame>world</odom_frame>
+      <robot_base_frame>base_link</robot_base_frame>
+      <odom_publish_frequency>50</odom_publish_frequency>
     </plugin>
   </gazebo>

File: src/bgr_description/urdf/bgr_ros2_control.xacro (robot description, xacro)
@@ -15,9 +15,9 @@
             </hardware>
         </xacro:unless>
-         <!-- Rear wheels: velocity-controlled by controllers -->
+         <!-- Rear wheels: effort-controlled by controllers -->
         <joint name="Wheel_rl_joint">
-            <command_interface name="velocity">
-              <param name="min">-100</param>
-              <param name="max">100</param>
+            <command_interface name="effort">
+              <param name="min">-241.5</param>
+              <param name="max">241.5</param>
             </command_interface>
             <state_interface name="position" />
@@ -25,7 +25,7 @@
         </joint>
         <joint name="Wheel_rr_joint">
-            <command_interface name="velocity">
-              <param name="min">-100</param>
-              <param name="max">100</param>
+            <command_interface name="effort">
+              <param name="min">-241.5</param>
+              <param name="max">241.5</param>
             </command_interface>
             <state_interface name="position" />
@@ -34,21 +34,24 @@
         <!-- Front steering and wheels -->
         <joint name="Steering_fl_joint">
-        <!-- Mimic joint: expose only state interfaces (no commands) -->
-        <state_interface name="position"/>
-        <state_interface name="velocity"/>
+            <command_interface name="position">
+                <param name="min">-0.384</param>
+                <param name="max">0.384</param>
+            </command_interface>
+            <state_interface name="position"/>
+            <state_interface name="velocity"/>
         </joint>
         <joint name="Steering_fr_joint">
-        <command_interface name="position">
-            <param name="min">-1</param>
-            <param name="max">1</param>
-        </command_interface>
-        <state_interface name="position"/>
-        <state_interface name="velocity"/>
+            <command_interface name="position">
+                <param name="min">-0.384</param>
+                <param name="max">0.384</param>
+            </command_interface>
+            <state_interface name="position"/>
+            <state_interface name="velocity"/>
         </joint>
-         <!-- Front wheels: velocity-controlled by controllers -->
+         <!-- Front wheels: effort-controlled by controllers -->
         <joint name="Wheel_fl_joint">
-        <command_interface name="velocity">
-            <param name="min">-100</param>
-            <param name="max">100</param>
+        <command_interface name="effort">
+            <param name="min">-241.5</param>
+              <param name="max">241.5</param>
         </command_interface>
         <state_interface name="position"/>
@@ -56,7 +59,7 @@
         </joint>
         <joint name="Wheel_fr_joint">
-        <command_interface name="velocity">
-            <param name="min">-100</param>
-            <param name="max">100</param>
+        <command_interface name="effort">
+            <param name="min">-241.5</param>
+              <param name="max">241.5</param>
         </command_interface>
         <state_interface name="position"/>

Commit message: IMU sensor addition

File: src/bgr_description/urdf/bgr.urdf.xacro (robot description, xacro)
@@ -187,3 +187,16 @@
     </collision>
   </link>
+  <!-- IMU -->
+  <joint name="imu_joint" type="fixed">
+    <origin xyz="0 0 0" rpy="0 0 0"/>
+    <parent link="base_link"/>
+    <child link="imu_link"/>
+  </joint>
+  <link name="imu_link">
+    <inertial>
+      <mass value="0.1"/>
+      <origin xyz="0 0 0" rpy="0 0 0"/>
+      <inertia ixx="0.00001" ixy="0" ixz="0" iyy="0.00001" iyz="0" izz="0.00001"/>
+    </inertial>
+  </link>
 </robot>

File: src/bgr_description/urdf/bgr_gazebo.xacro (robot description, xacro)
@@ -133,4 +133,13 @@
     </sensor>
   </gazebo>
+  <!-- IMU -->
+  <gazebo reference="imu_link">
+    <sensor name="imu_sensor" type="imu">
+      <always_on>true</always_on>
+      <update_rate>10</update_rate>
+      <visualize>true</visualize>
+      <topic>imu</topic>
+    </sensor>
+  </gazebo>
   <gazebo>
     <plugin filename="gz-sim-sensors-system" name="gz::sim::systems::Sensors">

Commit message: fix urdf bug missing parm

File: src/bgr_description/urdf/bgr.urdf.xacro (robot description, xacro)
@@ -203,4 +203,5 @@
   <link name="front_cam_link">
     <inertial>
+      <origin xyz="0 0 0" rpy="0 0 0"/>
       <mass value="0.01"/>
       <inertia ixx="0.001" ixy="0" ixz="0" iyy="0.001" iyz="0" izz="0.001"/>
