Commit message: Updated body mass, steer limit and wheel slip parameters for better simulation fidelity as well as adjusted keyboard teleop parameters for more precise control.

File: src/bgr_description/urdf/bgr.urdf.xacro (robot description, xacro)
@@ -14,6 +14,6 @@
   <xacro:property name="wheelbase"    value="2.0368"/>
    <!-- Mass and steering limits -->
-  <xacro:property name="body_mass"    value="50.0"/>
-  <xacro:property name="steer_limit"  value="0.6"/>
+  <xacro:property name="body_mass"    value="286.0"/>
+  <xacro:property name="steer_limit"  value="0.384"/>
   <!-- Bounding box used for base_link collision and inertia -->
   <xacro:property name="body_size_x"  value="2.0"/>

File: src/bgr_description/urdf/bgr_gazebo.xacro (robot description, xacro)
@@ -3,28 +3,28 @@
   <!-- Gazebo specific parameters -->
   <gazebo reference="Wheel_fl">
-    <mu1>1.2</mu1><mu2>1.2</mu2> <!-- coefficient of friction -->
+    <mu1>1</mu1><mu2>1</mu2> <!-- coefficient of friction -->
     <surface>
-      <friction><ode><mu>1.2</mu><mu2>1.2</mu2><slip1>0.01</slip1><slip2>0.01</slip2></ode></friction> <!-- friction parameters -->
+      <friction><ode><mu>1</mu><mu2>1</mu2><slip1>0.01</slip1><slip2>0.01</slip2></ode></friction> <!-- friction parameters -->
       <contact><ode><kp>1000000.0</kp><kd>1.0</kd><max_vel>0.1</max_vel><min_depth>0.001</min_depth></ode></contact> <!-- contact parameters -->
     </surface>
   </gazebo>
   <gazebo reference="Wheel_fr">
-    <mu1>1.2</mu1><mu2>1.2</mu2>
+    <mu1>1</mu1><mu2>1</mu2>
     <surface>
-      <friction><ode><mu>1.2</mu><mu2>1.2</mu2><slip1>0.01</slip1><slip2>0.01</slip2></ode></friction>
+      <friction><ode><mu>1</mu><mu2>1</mu2><slip1>0.01</slip1><slip2>0.01</slip2></ode></friction>
       <contact><ode><kp>1000000.0</kp><kd>1.0</kd><max_vel>0.1</max_vel><min_depth>0.001</min_depth></ode></contact>
     </surface>
   </gazebo>
   <gazebo reference="Wheel_rl">
-    <mu1>1.2</mu1><mu2>1.2</mu2>
+    <mu1>1</mu1><mu2>1</mu2>
     <surface>
-      <friction><ode><mu>1.2</mu><mu2>1.2</mu2><slip1>0.01</slip1><slip2>0.01</slip2></ode></friction>
+      <friction><ode><mu>1</mu><mu2>1</mu2><slip1>0.01</slip1><slip2>0.01</slip2></ode></friction>
       <contact><ode><kp>1000000.0</kp><kd>1.0</kd><max_vel>0.1</max_vel><min_depth>0.001</min_depth></ode></contact>
     </surface>
   </gazebo>
   <gazebo reference="Wheel_rr">
-    <mu1>1.2</mu1><mu2>1.2</mu2>
+    <mu1>1</mu1><mu2>1</mu2>
     <surface>
-      <friction><ode><mu>1.2</mu><mu2>1.2</mu2><slip1>0.01</slip1><slip2>0.01</slip2></ode></friction>
+      <friction><ode><mu>1</mu><mu2>1</mu2><slip1>0.01</slip1><slip2>0.01</slip2></ode></friction>
       <contact><ode><kp>1000000.0</kp><kd>1.0</kd><max_vel>0.1</max_vel><min_depth>0.001</min_depth></ode></contact>
     </surface>
@@ -67,18 +67,18 @@
     <plugin filename="gz-sim-wheel-slip-system" name="gz::sim::systems::WheelSlip">
       <wheel link_name="Wheel_rr">
-        <slip_compliance_lateral>0.05</slip_compliance_lateral>
-        <slip_compliance_longitudinal>0.001</slip_compliance_longitudinal>
+        <slip_compliance_lateral>0.0000333</slip_compliance_lateral>
+        <slip_compliance_longitudinal>0.0001</slip_compliance_longitudinal>
       </wheel>
       <wheel link_name="Wheel_rl">
-        <slip_compliance_lateral>0.05</slip_compliance_lateral>
-        <slip_compliance_longitudinal>0.001</slip_compliance_longitudinal>
+        <slip_compliance_lateral>0.0000333</slip_compliance_lateral>
+        <slip_compliance_longitudinal>0.0001</slip_compliance_longitudinal>
       </wheel>
       <wheel link_name="Wheel_fr">
-        <slip_compliance_lateral>0.05</slip_compliance_lateral>
-        <slip_compliance_longitudinal>0.001</slip_compliance_longitudinal>
+        <slip_compliance_lateral>0.0000333</slip_compliance_lateral>
+        <slip_compliance_longitudinal>0.0001</slip_compliance_longitudinal>
       </wheel>
       <wheel link_name="Wheel_fl">
-        <slip_compliance_lateral>0.05</slip_compliance_lateral>
-        <slip_compliance_longitudinal>0.001</slip_compliance_longitudinal>
+        <slip_compliance_lateral>0.0000333</slip_compliance_lateral>
+        <slip_compliance_longitudinal>0.0001</slip_compliance_longitudinal>
       </wheel>
     </plugin>

Commit message: Refactor build commands to remove --symlink-install and update URDF mesh file references; add new collision and visual mesh files for wheels and steering components.

File: src/bgr_description/urdf/bgr.urdf.xacro (robot description, xacro)
@@ -3,7 +3,4 @@
    <!-- Select Gazebo flavor (Ignition/GZ) to load the matching ros2_control hardware plugin -->
   <xacro:arg name="is_ignition" default="true"/>
-  <!-- External includes-->
-  <xacro:include filename="$(find bgr_description)/urdf/bgr_gazebo.xacro"/>
-  <xacro:include filename="$(find bgr_description)/urdf/bgr_ros2_control.xacro"/>
   <!-- === Basic params === -->
   <!-- Wheel geometry (radius/width) and chassis dimensions -->
@@ -20,4 +17,7 @@
   <xacro:property name="body_size_y"  value="1.0"/>
   <xacro:property name="body_size_z"  value="0.5"/>
+  <!-- External includes-->
+  <xacro:include filename="$(find bgr_description)/urdf/bgr_gazebo.xacro"/>
+  <xacro:include filename="$(find bgr_description)/urdf/bgr_ros2_control.xacro"/>
   <!-- === Base footprint === -->
   <link name="base_footprint"/>
@@ -42,5 +42,5 @@
       <origin xyz="0 0 0" rpy="0 0 0"/>
       <geometry>
-        <mesh filename="package://bgr_description/meshes/visual/base_link.STL"/>
+        <mesh filename="package://bgr_description/meshes/visual/base_link.stl"/>
       </geometry>
       <material name=""><color rgba="0.79216 0.81961 0.93333 1"/></material>
@@ -98,11 +98,11 @@
   <!-- === Wheels and Joints === -->
   <!-- rear wheels -->
-  <xacro:wheel_link name="Wheel_rl" visual_mesh="package://bgr_description/meshes/visual/Wheel_rl.STL"/>
-  <xacro:wheel_link name="Wheel_rr" visual_mesh="package://bgr_description/meshes/visual/Wheel_rr.STL"/>
+  <xacro:wheel_link name="Wheel_rl" visual_mesh="package://bgr_description/meshes/visual/Wheel_rl.stl"/>
+  <xacro:wheel_link name="Wheel_rr" visual_mesh="package://bgr_description/meshes/visual/Wheel_rr.stl"/>
   <!-- front wheels with steering stubs -->
   <xacro:stub_link name="Steering_fl"/>
-  <xacro:wheel_link name="Wheel_fl" visual_mesh="package://bgr_description/meshes/visual/Wheel_fl.STL"/>
+  <xacro:wheel_link name="Wheel_fl" visual_mesh="package://bgr_description/meshes/visual/Wheel_fl.stl"/>
   <xacro:stub_link name="Steering_fr"/>
-  <xacro:wheel_link name="Wheel_fr" visual_mesh="package://bgr_description/meshes/visual/Wheel_fr.STL"/>
+  <xacro:wheel_link name="Wheel_fr" visual_mesh="package://bgr_description/meshes/visual/Wheel_fr.stl"/>
   <!-- === Joints === -->
   <!-- rear left -->

File: src/bgr_description/urdf/bgr_gazebo.xacro (robot description, xacro)
@@ -69,16 +69,24 @@
         <slip_compliance_lateral>0.05</slip_compliance_lateral>
         <slip_compliance_longitudinal>0.001</slip_compliance_longitudinal>
+        <wheel_radius>${wheel_radius}</wheel_radius>
+        <wheel_normal_force>100</wheel_normal_force>
       </wheel>
       <wheel link_name="Wheel_rl">
         <slip_compliance_lateral>0.05</slip_compliance_lateral>
         <slip_compliance_longitudinal>0.001</slip_compliance_longitudinal>
+        <wheel_radius>${wheel_radius}</wheel_radius>
+        <wheel_normal_force>100</wheel_normal_force>
       </wheel>
       <wheel link_name="Wheel_fr">
         <slip_compliance_lateral>0.05</slip_compliance_lateral>
         <slip_compliance_longitudinal>0.001</slip_compliance_longitudinal>
+        <wheel_radius>${wheel_radius}</wheel_radius>
+        <wheel_normal_force>100</wheel_normal_force>
       </wheel>
       <wheel link_name="Wheel_fl">
         <slip_compliance_lateral>0.05</slip_compliance_lateral>
         <slip_compliance_longitudinal>0.001</slip_compliance_longitudinal>
+        <wheel_radius>${wheel_radius}</wheel_radius>
+        <wheel_normal_force>100</wheel_normal_force>
       </wheel>
     </plugin>

Commit message: Working version of simulator. Added GPS

File: src/bgr_description/urdf/bgr.urdf.xacro (robot description, xacro)
@@ -8,5 +8,5 @@
   <xacro:property name="track"        value="1.3092"/>
   <xacro:property name="wheelbase"    value="2.0368"/>
-   <!-- Mass and steering limits -->
+  <!-- Mass and steering limits -->
   <!-- Real measured total car mass is 283.6 kg. body_mass is the remaining
        base_link mass after separately modeled wheels, steering stubs, and sensors. -->
@@ -17,7 +17,13 @@
   <xacro:property name="imu_mass"           value="0.1"/>
   <xacro:property name="front_cam_mass"     value="0.01"/>
-  <xacro:property name="body_mass"          value="${total_vehicle_mass - (4*wheel_mass + 2*steering_stub_mass + lidar_mass + imu_mass + front_cam_mass)}"/>
+  <xacro:property name="gps_mass"           value="0.1"/>
+  <xacro:property name="body_mass"          value="${total_vehicle_mass - (4*wheel_mass + 2*steering_stub_mass + lidar_mass + imu_mass + front_cam_mass + gps_mass)}"/>
   <xacro:property name="wheel_normal_force" value="${total_vehicle_mass * 9.80665 / 4.0}"/>
   <xacro:property name="steer_limit"  value="0.6"/>
+  <!-- Sensor update rates (Hz) -->
+  <xacro:property name="lidar_update_rate"     value="50"/>
+  <xacro:property name="imu_update_rate"       value="10"/>
+  <xacro:property name="front_cam_update_rate" value="30"/>
+  <xacro:property name="gps_update_rate"       value="10"/>
   <!-- Mesh-bounds approximation used for base_link collision and inertia.
        Replace body_cg_* with measured CG values when available. -->
@@ -195,9 +201,4 @@
       </material>
     </visual>
-    <collision>
-      <geometry>
-        <cylinder radius="0.05" length="0.05"/>
-      </geometry>
-    </collision>
   </link>
   <!-- IMU -->
@@ -210,4 +211,17 @@
     <inertial>
       <mass value="${imu_mass}"/>
+      <origin xyz="0 0 0" rpy="0 0 0"/>
+      <inertia ixx="0.00001" ixy="0" ixz="0" iyy="0.00001" iyz="0" izz="0.00001"/>
+    </inertial>
+  </link>
+  <!-- GPS -->
+  <joint name="gps_joint" type="fixed">
+    <origin xyz="0.5 0 0.45" rpy="0 0 0"/>
+    <parent link="base_link"/>
+    <child link="gps_link"/>
+  </joint>
+  <link name="gps_link">
+    <inertial>
+      <mass value="${gps_mass}"/>
       <origin xyz="0 0 0" rpy="0 0 0"/>
       <inertia ixx="0.00001" ixy="0" ixz="0" iyy="0.00001" iyz="0" izz="0.00001"/>

File: src/bgr_description/urdf/bgr_gazebo.xacro (robot description, xacro)
@@ -104,5 +104,5 @@
       <always_on>false</always_on>
       <visualize>true</visualize>
-      <update_rate>50</update_rate>
+      <update_rate>${lidar_update_rate}</update_rate> <!-- Adjust in urdf -->
       <ray>
          <scan>
@@ -130,5 +130,5 @@
     <sensor name="imu_sensor" type="imu">
       <always_on>true</always_on>
-      <update_rate>10</update_rate>
+      <update_rate>${imu_update_rate}</update_rate> <!-- Adjust in urdf -->
       <visualize>true</visualize>
       <topic>/imu</topic>
@@ -146,5 +146,5 @@
       <always_on>false</always_on>
       <visualize>true</visualize>
-      <update_rate>30</update_rate>
+      <update_rate>${front_cam_update_rate}</update_rate> <!-- Adjust in urdf -->
       <topic>front_cam</topic>
       <camera>
@@ -162,4 +162,16 @@
     </sensor>
   </gazebo>
+  <!-- NavSat system plugin (Jazzy / gz-sim) -->
+  <gazebo>
+    <plugin filename="gz-sim-navsat-system" name="gz::sim::systems::NavSat"/>
+  </gazebo>
+  <!-- GPS (NavSat) Sensor -->
+  <gazebo reference="gps_link">
+    <sensor name="gps_sensor" type="navsat">
+      <always_on>true</always_on>
+      <update_rate>${gps_update_rate}</update_rate> <!-- Adjust in urdf -->
+      <topic>gps/fix</topic>
+    </sensor>
+  </gazebo>
   <!-- Sensor pipeline plugin (Jazzy / gz-sim) -->
   <gazebo>

Commit message: Reduced Camera, LiDAR Hz rate in Git Actions CI to improve RTF, configured GPS for worlds, visual cylinder on vehicle and added a test for it in the test_simultion

File: src/bgr_description/urdf/bgr.urdf.xacro (robot description, xacro)
@@ -22,7 +22,9 @@
   <xacro:property name="steer_limit"  value="0.6"/>
   <!-- Sensor update rates (Hz) -->
-  <xacro:property name="lidar_update_rate"     value="50"/>
+  <xacro:arg name="lidar_update_rate"     default="50"/>
+  <xacro:arg name="front_cam_update_rate" default="30"/>
+  <xacro:property name="lidar_update_rate"     value="$(arg lidar_update_rate)"/>
   <xacro:property name="imu_update_rate"       value="10"/>
-  <xacro:property name="front_cam_update_rate" value="30"/>
+  <xacro:property name="front_cam_update_rate" value="$(arg front_cam_update_rate)"/>
   <xacro:property name="gps_update_rate"       value="10"/>
   <!-- Mesh-bounds approximation used for base_link collision and inertia.
@@ -227,4 +229,12 @@
       <inertia ixx="0.00001" ixy="0" ixz="0" iyy="0.00001" iyz="0" izz="0.00001"/>
     </inertial>
+    <visual>
+      <geometry>
+        <cylinder radius="0.04" length="0.02"/>
+      </geometry>
+      <material name="orange">
+        <color rgba="1.0 0.5 0.0 1.0"/>
+      </material>
+    </visual>
   </link>
   <!-- Front Camera - To run: ros2 run rqt_image_view rqt_image_view after launching gazebo -->
